Commit message: 加入cdut_dog模型

File: dog_bringup/xacro/cdut_dog/dog.urdf (robot description, URDF)
Before this commit: robot dog, 19 links, 18 joints
Links:
- link LF_FOOT: mass 0.06 -> 0.059
- link LF_HIP: mass 0.55 -> 0.53; geometry visual mesh filename=package://dog_bringup/meshes/cdut_dog/hip.STL scale=1 1 1
- link LF_SHANK: mass 0.153 -> 0.084; geometry collision cylinder length=0.10 radius=0.015; collision cylinder length=0.12 radius=0.015
- link LF_THIGH: mass 0.86 -> 0.75; geometry collision box size=0.04 0.045 0.2; visual mesh filename=package://dog_bringup/meshes/cdut_dog/thigh.STL scale=1 1 1
- link LH_FOOT: mass 0.06 -> 0.059
- link LH_HIP: mass 0.55 -> 0.53; geometry visual mesh filename=package://dog_bringup/meshes/cdut_dog/hip.STL scale=-1 1 1
- link LH_SHANK: mass 0.153 -> 0.084; geometry collision cylinder length=0.10 radius=0.015; collision cylinder length=0.12 radius=0.015
- link LH_THIGH: mass 0.86 -> 0.75; geometry collision box size=0.04 0.045 0.2; visual mesh filename=package://dog_bringup/meshes/cdut_dog/thigh.STL scale=1 1 1
- link RF_FOOT: mass 0.06 -> 0.059
- link RF_HIP: mass 0.55 -> 0.53; geometry visual mesh filename=package://dog_bringup/meshes/cdut_dog/hip.STL scale=1 -1 1
- link RF_SHANK: mass 0.153 -> 0.084; geometry collision cylinder length=0.10 radius=0.015; collision cylinder length=0.12 radius=0.015
- link RF_THIGH: mass 0.86 -> 0.75; geometry collision box size=0.04 0.045 0.2; visual mesh filename=package://dog_bringup/meshes/cdut_dog/thigh.STL scale=1 -1 1
- link RH_FOOT: mass 0.06 -> 0.059
- link RH_HIP: mass 0.55 -> 0.53; geometry visual mesh filename=package://dog_bringup/meshes/cdut_dog/hip.STL scale=-1 -1 1
- link RH_SHANK: mass 0.153 -> 0.084; geometry collision cylinder length=0.10 radius=0.015; collision cylinder length=0.12 radius=0.015
- link RH_THIGH: mass 0.86 -> 0.75; geometry collision box size=0.04 0.045 0.2; visual mesh filename=package://dog_bringup/meshes/cdut_dog/thigh.STL scale=1 -1 1
- link TORSO: mass 5.6056 -> 5.35; geometry collision box size=0.25 0.232 0.11; visual mesh filename=package://dog_bringup/meshes/cdut_dog/torso.STL
Joints:
- joint LF_Ankle: origin xyz=0 0 -0.21012 -> xyz=0.183238 0.002132 -0.125966
- joint LF_HAA: limit lower=-0.523 upper=0.523 effort=24 velocity=26.2 -> lower=-0.5 upper=0.5 effort=24 velocity=26.2; origin xyz=0.1745 0.062 0 -> xyz=0.12556 0.06752 0.007
- joint LF_HFE: limit lower=-2.67 upper=0.314 effort=24 velocity=26.2 -> lower=-2 upper=1.6 effort=24 velocity=26.2; origin xyz=0 0.09735 0 -> xyz=0.0485 0.004 0
- joint LF_KFE: limit lower=0.524 upper=2.792 effort=36 velocity=17.3 -> lower=-2 upper=0.5 effort=36 velocity=17.3; origin xyz=0 0 -0.2 -> xyz=-0.176118 0.09439 -0.09319
- joint LH_Ankle: origin xyz=0 0 -0.21012 -> xyz=0.183238 0.002132 -0.125966
- joint LH_HAA: limit lower=-0.523 upper=0.523 effort=24 velocity=26.2 -> lower=-0.5 upper=0.5 effort=24 velocity=26.2; origin xyz=-0.1745 0.062 0 -> xyz=-0.12556 0.06752 0.007
- joint LH_HFE: limit lower=-2.67 upper=0.314 effort=24 velocity=26.2 -> lower=-2 upper=1.6 effort=24 velocity=26.2; origin xyz=0 0.09735 0 -> xyz=-0.0485 0.004 0
- joint LH_KFE: limit lower=0.524 upper=2.792 effort=36 velocity=17.3 -> lower=-2 upper=0.5 effort=36 velocity=17.3; origin xyz=0 0 -0.2 -> xyz=-0.176118 0.09439 -0.09319
- joint RF_Ankle: origin xyz=0 0 -0.21012 -> xyz=0.183238 -0.002132 -0.125966
- joint RF_HAA: limit lower=-0.523 upper=0.523 effort=24 velocity=26.2 -> lower=-0.5 upper=0.5 effort=24 velocity=26.2; origin xyz=0.1745 -0.062 0 -> xyz=0.12556 -0.06752 0.007
- joint RF_HFE: limit lower=-2.67 upper=0.314 effort=24 velocity=26.2 -> lower=-2 upper=1.6 effort=24 velocity=26.2; origin xyz=0 -0.09735 0 -> xyz=0.0485 -0.004 0
- joint RF_KFE: limit lower=0.524 upper=2.792 effort=36 velocity=17.3 -> lower=-2 upper=0.5 effort=36 velocity=17.3; origin xyz=0 0 -0.2 -> xyz=-0.176118 -0.09439 -0.09319
- joint RH_Ankle: origin xyz=0 0 -0.21012 -> xyz=0.183238 -0.002132 -0.125966
- joint RH_HAA: limit lower=-0.523 upper=0.523 effort=24 velocity=26.2 -> lower=-0.5 upper=0.5 effort=24 velocity=26.2; origin xyz=-0.1745 -0.062 0 -> xyz=-0.12556 -0.06752 0.007
- joint RH_HFE: limit lower=-2.67 upper=0.314 effort=24 velocity=26.2 -> lower=-2 upper=1.6 effort=24 velocity=26.2; origin xyz=0 -0.09735 0 -> xyz=-0.0485 -0.004 0
- joint RH_KFE: limit lower=0.524 upper=2.792 effort=36 velocity=17.3 -> lower=-2 upper=0.5 effort=36 velocity=17.3; origin xyz=0 0 -0.2 -> xyz=-0.176118 -0.09439 -0.09319

File: dog_bringup/xacro/lite3/const.xacro (robot description, xacro)
@@ -2,5 +2,5 @@
 <robot xmlns:xacro="http://www.ros.org/wiki/xacro">
     <!-- xacro ./dog.xacro > dog.urdf -->
-    <xacro:property name="mesh_path" value="package://dog_bringup/meshes"/>
+    <xacro:property name="mesh_path" value="package://dog_bringup/meshes/lite3"/>
     <xacro:property name="cfg" value="${xacro.load_yaml('$(find dog_bringup)/config/robot_controllers.yaml')}"/>
 <!-- 躯干参数 -->
