Commit message: 增加J60驱动

File: dog_bringup/xacro/cdut_dog/const.xacro (robot description, xacro)
@@ -3,5 +3,5 @@
     <!-- xacro ./dog.xacro > dog.urdf -->
     <xacro:property name="mesh_path" value="package://dog_bringup/meshes/cdut_dog"/>
-    <xacro:property name="cfg" value="${xacro.load_yaml('$(find dog_bringup)/config/robot_controllers.yaml')}"/>
+    <xacro:property name="cfg" value="${xacro.load_yaml('$(find dog_bringup)/config/cdut_dog/robot_controllers.yaml')}"/>
 <!-- 躯干参数 -->
 <xacro:property name="torso_mass" value="5.35"/>        <!-- 躯干质量(kg) -->
@@ -64,14 +64,14 @@
 <xacro:property name="hipx_max" value="0.5"/>           <!-- 髋x轴关节最大角度(rad，约30°) -->
 <xacro:property name="hipx_vel" value="26.2"/>            <!-- 髋x轴关节最大角速度(rad/s) -->
-<xacro:property name="hipx_eff" value="24"/>              <!-- 髋x轴关节最大力矩(N·m) -->
+<xacro:property name="hipx_eff" value="12"/>              <!-- 髋x轴关节最大力矩(N·m) -->
 <!-- 髋关节y轴关节限位&性能参数 -->
 <xacro:property name="hipy_min" value="-2"/>           <!-- 髋y轴关节最小角度(rad) -->
 <xacro:property name="hipy_max" value="1.6"/>           <!-- 髋y轴关节最大角度(rad，约18°) -->
 <xacro:property name="hipy_vel" value="26.2"/>            <!-- 髋y轴关节最大角速度(rad/s) -->
-<xacro:property name="hipy_eff" value="24"/>              <!-- 髋y轴关节最大力矩(N·m) -->
+<xacro:property name="hipy_eff" value="12"/>              <!-- 髋y轴关节最大力矩(N·m) -->
 <!-- 膝关节限位&性能参数 -->
 <xacro:property name="knee_min" value="-2"/>           <!-- 膝关节最小角度(rad，约30°) -->
 <xacro:property name="knee_max" value="0.5"/>           <!-- 膝关节最大角度(rad，约160°) -->
 <xacro:property name="knee_vel" value="17.3"/>            <!-- 膝关节最大角速度(rad/s) -->
-<xacro:property name="knee_eff" value="36"/>              <!-- 膝关节最大力矩(N·m) -->
+<xacro:property name="knee_eff" value="12"/>              <!-- 膝关节最大力矩(N·m) -->
 </robot>

File: dog_bringup/xacro/cdut_dog/dog.urdf (robot description, URDF)
Before this commit: robot dog, 19 links, 18 joints
Links:
- added link lidar_link, mass 0.24; visual mesh filename=package://dog_bringup/meshes/cdut_dog/MID360.STL
Joints:
- added joint lidar_joint: type fixed, parent base_link, child lidar_link, origin xyz=0.15556 0.0005199 0.13105, axis 0 0 0

File: dog_bringup/xacro/cdut_dog/dog.xacro (robot description, xacro)
@@ -43,4 +43,33 @@
         <origin xyz="0 0 0" rpy="0 0 0"/>
     </joint>
+    <!-- <link
+    name="lidar_link">
+    <inertial>
+      <origin
+        xyz="3.33066907387547E-15 9.9475983006414E-14 -0.0268465534683788"
+        rpy="0 0 0" />
+      <mass value="0.24" />
+      <inertia
+        ixx="0.000132876366974801"
+        ixy="2.45046624096634E-19"
+        ixz="-1.10460624029042E-19"
+        iyy="0.000108720544937996"
+        iyz="-8.27219261425137E-17"
+        izz="0.000193942390461225" />
+    </inertial>
+    <visual>
+      <origin xyz="0 0 0" rpy="0 0 0" />
+      <geometry>
+        <mesh
+          filename="${mesh_path}/MID360.STL" />
+      </geometry>
+    </visual>
+  </link>
+  <joint name="lidar_joint" type="fixed">
+    <origin xyz="0.15556 0.0005199 0.13105" />
+    <parent link="base_link" />
+    <child link="lidar_link" />
+    <axis xyz="0 0 0" />
+  </joint> -->
     <xacro:dog_leg name="LF" mirror="1" f_b="1"/>
     <xacro:dog_leg name="LH" mirror="1" f_b="-1"/>
@@ -49,10 +78,7 @@
     <ros2_control name="dog_System" type="system">
         <hardware>
-            <!-- <plugin>gazebo_ros2_control/GazeboSystem</plugin> -->
-            <plugin>dog_hardware/DogGazeboHW</plugin>
-            <param name="delay">${cfg['controller_manager']['ros__parameters']['hw_params']['delay']}</param>
-            <param name="imu_accel_var">${cfg['controller_manager']['ros__parameters']['imu_params']['accel']['variance']}</param>
-            <param name="imu_gyro_var">${cfg['controller_manager']['ros__parameters']['imu_params']['gyro']['variance']}</param>
-            <param name="imu_ori_var">${cfg['controller_manager']['ros__parameters']['imu_params']['orientation']['variance']}</param>
+            <!-- <plugin>dog_hardware/DogGazeboHW</plugin>
+            <param name="delay">${cfg['controller_manager']['ros__parameters']['hw_params']['delay']}</param> -->
+            <plugin>dog_hardware/J60_6_hw</plugin>
         </hardware>
         <sensor name="imu_sensor">
@@ -67,7 +93,4 @@
             <state_interface name="linear_acceleration.y"/>
             <state_interface name="linear_acceleration.z"/>
-            <state_interface name="orientation_covariance"/>
-            <state_interface name="angular_velocity_covariance"/>
-            <state_interface name="linear_acceleration_covariance"/>
         </sensor>
         <sensor name="LF_contact_sensor"> <state_interface name="contact"/></sensor>
@@ -84,26 +107,9 @@
         <always_on>true</always_on>
         <update_rate>1000</update_rate>
-        <imu>
-          <orientation>
-            <x><noise type="gaussian"><stddev>${cfg['controller_manager']['ros__parameters']['imu_params']['orientation']['variance']**0.5}</stddev></noise></x>
-            <y><noise type="gaussian"><stddev>${cfg['controller_manager']['ros__parameters']['imu_params']['orientation']['variance']**0.5}</stddev></noise></y>
-            <z><noise type="gaussian"><stddev>${cfg['controller_manager']['ros__parameters']['imu_params']['orientation']['variance']**0.5}</stddev></noise></z>
-          </orientation>
-          <linear_acceleration>
-            <x><noise type="gaussian"><stddev>${cfg['controller_manager']['ros__parameters']['imu_params']['accel']['variance']**0.5}</stddev><bias_mean>${cfg['controller_manager']['ros__parameters']['imu_params']['accel']['bias_mean']}</bias_mean></noise></x>
-            <y><noise type="gaussian"><stddev>${cfg['controller_manager']['ros__parameters']['imu_params']['accel']['variance']**0.5}</stddev><bias_mean>${cfg['controller_manager']['ros__parameters']['imu_params']['accel']['bias_mean']}</bias_mean></noise></y>
-            <z><noise type="gaussian"><stddev>${cfg['controller_manager']['ros__parameters']['imu_params']['accel']['variance']**0.5}</stddev><bias_mean>${cfg['controller_manager']['ros__parameters']['imu_params']['accel']['bias_mean']}</bias_mean></noise></z>
-          </linear_acceleration>
-          <angular_velocity>
-            <x><noise type="gaussian"><stddev>${cfg['controller_manager']['ros__parameters']['imu_params']['gyro']['variance']**0.5}</stddev><bias_mean>${cfg['controller_manager']['ros__parameters']['imu_params']['gyro']['bias_mean']}</bias_mean></noise></x>
-            <y><noise type="gaussian"><stddev>${cfg['controller_manager']['ros__parameters']['imu_params']['gyro']['variance']**0.5}</stddev><bias_mean>${cfg['controller_manager']['ros__parameters']['imu_params']['gyro']['bias_mean']}</bias_mean></noise></y>
-            <z><noise type="gaussian"><stddev>${cfg['controller_manager']['ros__parameters']['imu_params']['gyro']['variance']**0.5}</stddev><bias_mean>${cfg['controller_manager']['ros__parameters']['imu_params']['gyro']['bias_mean']}</bias_mean></noise></z>
-          </angular_velocity>
-        </imu>
       </sensor>
     </gazebo>
     <gazebo>
         <plugin filename="libgazebo_ros2_control.so" name="gazebo_ros2_control">
-            <parameters>$(find dog_bringup)/config/robot_controllers.yaml</parameters>
+            <parameters>$(find dog_bringup)/config/cdut_dog/robot_controllers.yaml</parameters>
             <robot_param>robot_description</robot_param>
             <robot_param_node>robot_state_publisher</robot_param_node>

File: dog_bringup/xacro/cdut_dog/ros2_control.xacro (robot description, xacro)
@@ -11,5 +11,4 @@
             <command_interface name="kp"/>
             <command_interface name="kd"/>
-            <command_interface name="mode"/>
             <state_interface name="driver_tem"/>
             <state_interface name="motor_tem"/>
@@ -28,5 +27,4 @@
             <command_interface name="kp"/>
             <command_interface name="kd"/>
-            <command_interface name="mode"/>
             <state_interface name="driver_tem"/>
             <state_interface name="motor_tem"/>
@@ -45,5 +43,4 @@
             <command_interface name="kp"/>
             <command_interface name="kd"/>
-            <command_interface name="mode"/>
             <state_interface name="driver_tem"/>
             <state_interface name="motor_tem"/>

File: dog_bringup/xacro/lite3/const.xacro (robot description, xacro)
@@ -3,5 +3,5 @@
     <!-- xacro ./dog.xacro > dog.urdf -->
     <xacro:property name="mesh_path" value="package://dog_bringup/meshes/lite3"/>
-    <xacro:property name="cfg" value="${xacro.load_yaml('$(find dog_bringup)/config/robot_controllers.yaml')}"/>
+    <xacro:property name="cfg" value="${xacro.load_yaml('$(find dog_bringup)/config/lite3/robot_controllers.yaml')}"/>
 <!-- 躯干参数 -->
 <xacro:property name="torso_mass" value="5.6056"/>        <!-- 躯干质量(kg) -->

File: dog_bringup/xacro/lite3/dog.xacro (robot description, xacro)
@@ -111,5 +111,5 @@
     <gazebo>
         <plugin filename="libgazebo_ros2_control.so" name="gazebo_ros2_control">
-            <parameters>$(find dog_bringup)/config/robot_controllers.yaml</parameters>
+            <parameters>$(find dog_bringup)/config/lite3/robot_controllers.yaml</parameters>
             <robot_param>robot_description</robot_param>
             <robot_param_node>robot_state_publisher</robot_param_node>

Commit message: 站立

File: dog_bringup/xacro/cdut_dog/const.xacro (robot description, xacro)
@@ -74,4 +74,4 @@
 <xacro:property name="knee_max" value="0.5"/>           <!-- 膝关节最大角度(rad，约160°) -->
 <xacro:property name="knee_vel" value="17.3"/>            <!-- 膝关节最大角速度(rad/s) -->
-<xacro:property name="knee_eff" value="12"/>              <!-- 膝关节最大力矩(N·m) -->
+<xacro:property name="knee_eff" value="30"/>              <!-- 膝关节最大力矩(N·m) -->
 </robot>

File: dog_bringup/xacro/cdut_dog/dog.xacro (robot description, xacro)
@@ -1,4 +1,5 @@
 <?xml version="1.0"?>
 <robot name="dog" xmlns:xacro="http://www.ros.org/wiki/xacro">
+    <xacro:arg name="is_sim" default="true"/>
     <xacro:include filename="./const.xacro"/>
     <xacro:include filename="./ros2_control.xacro"/>
@@ -78,7 +79,11 @@
     <ros2_control name="dog_System" type="system">
         <hardware>
-            <!-- <plugin>dog_hardware/DogGazeboHW</plugin>
-            <param name="delay">${cfg['controller_manager']['ros__parameters']['hw_params']['delay']}</param> -->
-            <plugin>dog_hardware/J60_6_hw</plugin>
+            <xacro:if value="$(arg is_sim)">
+                <plugin>dog_hardware/DogGazeboHW</plugin>
+                <param name="delay">${cfg['controller_manager']['ros__parameters']['hw_params']['delay']}</param>
+            </xacro:if>
+            <xacro:unless value="$(arg is_sim)">
+                <plugin>dog_hardware/J60_6_hw</plugin>
+            </xacro:unless>
         </hardware>
         <sensor name="imu_sensor">
@@ -103,29 +108,31 @@
         <xacro:leg_control_interface name="RH"/>
     </ros2_control>
-    <gazebo reference="imu_link">
-      <sensor name="imu_sensor" type="imu">
-        <always_on>true</always_on>
-        <update_rate>1000</update_rate>
-      </sensor>
-    </gazebo>
-    <gazebo>
-        <plugin filename="libgazebo_ros2_control.so" name="gazebo_ros2_control">
-            <parameters>$(find dog_bringup)/config/cdut_dog/robot_controllers.yaml</parameters>
-            <robot_param>robot_description</robot_param>
-            <robot_param_node>robot_state_publisher</robot_param_node>
-        </plugin>
-    </gazebo>
-    <gazebo>
-      <plugin name="dog_ground_truth" filename="libgazebo_ros_p3d.so">
-        <ros>
-          <remapping>odom:=/ground_truth</remapping>
-        </ros>
-        <body_name>base_link</body_name>
-        <frame_name>world</frame_name>
-        <update_rate>10.0</update_rate>
-        <xyz_offset>0 0 0</xyz_offset>
-        <rpy_offset>0 0 0</rpy_offset>
-        <gaussian_noise>0.001</gaussian_noise>
-      </plugin>
-    </gazebo>
+    <xacro:if value="$(arg is_sim)">
+        <gazebo reference="imu_link">
+          <sensor name="imu_sensor" type="imu">
+            <always_on>true</always_on>
+            <update_rate>1000</update_rate>
+          </sensor>
+        </gazebo>
+        <gazebo>
+            <plugin filename="libgazebo_ros2_control.so" name="gazebo_ros2_control">
+                <parameters>$(find dog_bringup)/config/cdut_dog/robot_controllers.yaml</parameters>
+                <robot_param>robot_description</robot_param>
+                <robot_param_node>robot_state_publisher</robot_param_node>
+            </plugin>
+        </gazebo>
+        <gazebo>
+          <plugin name="dog_ground_truth" filename="libgazebo_ros_p3d.so">
+            <ros>
+              <remapping>odom:=/ground_truth</remapping>
+            </ros>
+            <body_name>base_link</body_name>
+            <frame_name>world</frame_name>
+            <update_rate>10.0</update_rate>
+            <xyz_offset>0 0 0</xyz_offset>
+            <rpy_offset>0 0 0</rpy_offset>
+            <gaussian_noise>0.001</gaussian_noise>
+          </plugin>
+        </gazebo>
+    </xacro:if>
 </robot>
